File: RGB_LED_CONTROLLER-HP/RGB_LED_CONTROLLER-HP.sch (KiCad schematic (older format))
At the start: 25 parts, among them J1 PWR IN, J2 PWM OUT, J3 AUX, Q1 IRF540N, Q2 IRF540N, Q3 IRF540N, SW1 SW_Push, U1 PIC12F629-IP, U1 PIC12F675-IP, U2 LM78L05_TO92

Commit message: Second Commit
Parts:
- removed D1: 1N4148, Diode_THT:D_DO-35_SOD27_P7.62mm_Horizontal, symbol Diode:1N4148
- removed J1: PWR IN, symbol Connector:Screw_Terminal_01x02
- removed J2: PWM OUT, symbol Connector:Screw_Terminal_01x04
- removed R? (x2): 10K, symbol Device:R
- removed U1: PIC12F675-IP, Package_DIP:DIP-8_W7.62mm, symbol MCU_Microchip_PIC12:PIC12F675-IP
- added C3: 10uF 10V, Capacitor_THT:CP_Radial_D5.0mm_P2.50mm, symbol Device:CP
- added D1: 1N4001, Diode_THT:D_DO-41_SOD81_P10.16mm_Horizontal, symbol Diode:1N4001
- added J1: Terminal Block, symbol Connector:Screw_Terminal_01x05
- added R7, R8: 10K, Resistor_THT:R_Axial_DIN0207_L6.3mm_D2.5mm_P10.16mm_Horizontal, symbol Device:R
- added R9: 100R, Resistor_THT:R_Axial_DIN0207_L6.3mm_D2.5mm_P10.16mm_Horizontal, symbol Device:R
- C1: footprint (none) -> Capacitor_THT:CP_Radial_D8.0mm_P3.50mm
- C2: footprint (none) -> Capacitor_THT:C_Disc_D3.0mm_W1.6mm_P2.50mm
- H1, H2, H3, H4: footprint (none) -> MountingHole:MountingHole_2.7mm_M2.5
- J2: renamed from J3; footprint (none) -> Connector_PinHeader_2.54mm:PinHeader_1x03_P2.54mm_Vertical
- R1, R2, R3, R4, R5, R6: renamed from R?; footprint (none) -> Resistor_THT:R_Axial_DIN0207_L6.3mm_D2.5mm_P10.16mm_Horizontal
- SW1: footprint (none) -> Button_Switch_THT:SW_Tactile_SPST_Angled_PTS645Vx83-2LFS
Connections:
- net +5V: now reaches U1.1 (VDD)
- net +5V: now also C2.1, R1.1, R2.1, U2.1 (VO), R9.1
- net at U1.2 (GP5): now also R2.2, SW1.2
- net at U1.3 (GP4): now also R5.1
- net at U1.4 (GP3): now also R1.2
- net AUX: now reaches U1.5 (GP2)
- net AUX: now also J2.1 (Pin_1)
- net at U1.6 (GP1): now also R4.1
- net at U1.7 (GP0): now also R3.1
- net GND: now reaches U1.8 (VSS)
- net GND: now also C1.2, C2.2, J2.2 (Pin_2), Q1.3 (S), Q2.3 (S), Q3.3 (S), R6.2, SW1.1, U2.2 (GND), C3.2, J1.5 (Pin_5), R7.2, R8.2
- net at C1.1: now also U2.3 (VI), D1.1 (K)
- net at J2.3 (Pin_3): now also C3.1, R9.2
- net at Q2.1 (G): now also R4.2, R7.1
- net GREEN: now reaches Q2.2 (D)
- net GREEN: now also J1.2 (Pin_2)
- net at Q1.1 (G): now also R3.2, R6.1
- net RED: now reaches Q1.2 (D)
- net RED: now also J1.1 (Pin_1)
- net at Q3.1 (G): now also R5.2, R8.1
- net BLUE: now reaches Q3.2 (D)
- net BLUE: now also J1.3 (Pin_3)
- new net +12V: D1.2 (A), J1.4 (Pin_4)
Other:
- note added: "TSOP4838 IR RECEIVER\nNOT REQUIRED"
- moved on the sheet: C1, C2, H3, J2, Q1, Q2, Q3, R1, R2, R3, R4, R5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

Commit message: added custom footprint
Parts:
- removed Q1, Q2, Q3: IRF540N, Package_TO_SOT_THT:TO-220-3_Vertical, symbol Transistor_FET:IRF540N
- added Q1, Q2, Q3: IRLZ44N, Package_TO_SOT_THT:TO-220-3_Vertical, symbol Transistor_FET:IRLZ44N
- J1: footprint (none) -> Barrier_Terminal_Block_TE-Connectivity:Barrier_Terminal_Block_TE_4DB-P108-05_5P_8.26mm
- R3, R4, R5: value 120R -> 150R
- renumbered C2 to C1, C1 to C2
Connections:
- net +12V: now also J1.2 (Pin_2); no longer J1.4 (Pin_4)
- net BLUE: now also Q3.2 (D)
- net GND: now also J1.1 (Pin_1), Q1.3 (S), Q2.3 (S), Q3.3 (S); no longer J1.5 (Pin_5)
- net GREEN: now also J1.4 (Pin_4), Q2.2 (D); no longer J1.2 (Pin_2)
- net RED: now also J1.5 (Pin_5), Q1.2 (D); no longer J1.1 (Pin_1)
- net at R4.2, R7.1: now also Q2.1 (G)
- net at R3.2, R6.1: now also Q1.1 (G)
- net at R5.2, R8.1: now also Q3.1 (G)
Other:
- note added: "IRLZ44NPBF - LOGIC LEVEL N-CHANNEL MOSFET\nQ1 RED\nQ2GREEN\nQ3BLUE"
- note removed: "Q1 RED\nQ2GREEN\nQ3BLUE"
Changed lines of the file:
@@
 $EndComp
 $Comp
-L Device:CP C1
+L Device:CP C2
 U 1 1 6348DF12
 P 3060 2060
-F 0 "C1" H 2800 2110 50  0000 L CNN
+F 0 "C2" H 2800 2110 50  0000 L CNN
 F 1 "100uF 25V" H 2520 2000 50  0000 L CNN
 F 2 "Capacitor_THT:CP_Radial_D8.0mm_P3.50mm" H 3098 1910 50  0001 C CNN
@@
 $EndComp
 $Comp
-L Device:C C2
+L Device:C C1
 U 1 1 6348E200
 P 4090 2060
-F 0 "C2" H 4205 2106 50  0000 L CNN
+F 0 "C1" H 4205 2106 50  0000 L CNN
 F 1 "100nF" H 4205 2015 50  0000 L CNN
 F 2 "Capacitor_THT:C_Disc_D3.0mm_W1.6mm_P2.50mm" H 4128 1910 50  0001 C CNN
@@
 F 3 "~" H 4180 6450 50  0001 C CNN
 	1    4180 6450
-	1    0    0    -1
-$EndComp
-$Comp
-L Transistor_FET:IRF540N Q2
-U 1 1 63491091
-P 7140 3820
-F 0 "Q2" H 7346 3866 50  0000 L CNN
-F 1 "IRF540N" H 7346 3775 50  0000 L CNN
-F 2 "Package_TO_SOT_THT:TO-220-3_Vertical" H 7390 3745 50  0001 L CIN
-F 3 "http://www.irf.com/product-info/datasheets/data/irf540n.pdf" H 7140 3820 50  0001 L CNN
-	1    7140 3820
-	1    0    0    -1
-$EndComp
-$Comp
-L Transistor_FET:IRF540N Q1
-U 1 1 63491B6D
-P 6500 3160
-F 0 "Q1" H 6706 3206 50  0000 L CNN
-F 1 "IRF540N" H 6706 3115 50  0000 L CNN
-F 2 "Package_TO_SOT_THT:TO-220-3_Vertical" H 6750 3085 50  0001 L CIN
-F 3 "http://www.irf.com/product-info/datasheets/data/irf540n.pdf" H 6500 3160 50  0001 L CNN
-	1    6500 3160
-	1    0    0    -1
-$EndComp
-$Comp
-L Transistor_FET:IRF540N Q3
-U 1 1 63492175
-P 7850 4490
-F 0 "Q3" H 8056 4536 50  0000 L CNN
-F 1 "IRF540N" H 8056 4445 50  0000 L CNN
-F 2 "Package_TO_SOT_THT:TO-220-3_Vertical" H 8100 4415 50  0001 L CIN
-F 3 "http://www.irf.com/product-info/datasheets/data/irf540n.pdf" H 7850 4490 50  0001 L CNN
-	1    7850 4490
 	1    0    0    -1
 $EndComp
@@
 U 1 1 634930DF
 P 5720 4490
-F 0 "R5" H 5790 4536 50  0000 L CNN
-F 1 "120R" H 5790 4445 50  0000 L CNN
+F 0 "R5" V 5890 4440 50  0000 L CNN
+F 1 "150R" V 5810 4390 50  0000 L CNN
 F 2 "Resistor_THT:R_Axial_DIN0207_L6.3mm_D2.5mm_P10.16mm_Horizontal" V 5650 4490 50  0001 C CNN
 F 3 "~" H 5720 4490 50  0001 C CNN
@@
 U 1 1 63493C04
 P 5720 3820
-F 0 "R4" H 5790 3866 50  0000 L CNN
-F 1 "120R" H 5790 3775 50  0000 L CNN
+F 0 "R4" V 5890 3770 50  0000 L CNN
+F 1 "150R" V 5810 3720 50  0000 L CNN
 F 2 "Resistor_THT:R_Axial_DIN0207_L6.3mm_D2.5mm_P10.16mm_Horizontal" V 5650 3820 50  0001 C CNN
 F 3 "~" H 5720 3820 50  0001 C CNN
@@
 U 1 1 63494056
 P 5720 3160
-F 0 "R3" H 5790 3206 50  0000 L CNN
-F 1 "120R" H 5790 3115 50  0000 L CNN
+F 0 "R3" V 5890 3110 50  0000 L CNN
+F 1 "150R" V 5810 3060 50  0000 L CNN
 F 2 "Resistor_THT:R_Axial_DIN0207_L6.3mm_D2.5mm_P10.16mm_Horizontal" V 5650 3160 50  0001 C CNN
 F 3 "~" H 5720 3160 50  0001 C CNN
@@
 	1    0    0    -1
 $EndComp
-Text Notes 5160 2680 0    79   ~ 0
-Q1 RED\nQ2GREEN\nQ3BLUE
+Text Notes 5800 2320 0    79   ~ 0
+IRLZ44NPBF - LOGIC LEVEL N-CHANNEL MOSFET\nQ1 RED\nQ2GREEN\nQ3BLUE
 $Comp
 L Connector:Screw_Terminal_01x05 J1
@@
 F 0 "J1" H 9170 4212 50  0000 L CNN
 F 1 "Terminal Block" H 9170 4121 50  0000 L CNN
-F 2 "" H 9090 4170 50  0001 C CNN
+F 2 "Barrier_Terminal_Block_TE-Connectivity:Barrier_Terminal_Block_TE_4DB-P108-05_5P_8.26mm" H 9090 4170 50  0001 C CNN
 F 3 "~" H 9090 4170 50  0001 C CNN
 	1    9090 4170
-	1    0    0    -1
+	1    0    0    1
 $EndComp
 $Comp
@@
 Wire Wire Line
 	6600 2840 8640 2840
+$Comp
+L Transistor_FET:IRLZ44N Q1
+U 1 1 63FBD871
+P 6500 3160
+F 0 "Q1" H 6705 3207 50  0000 L CNN
+F 1 "IRLZ44N" H 6705 3114 50  0000 L CNN
+F 2 "Package_TO_SOT_THT:TO-220-3_Vertical" H 6750 3085 50  0001 L CIN
+F 3 "http://www.irf.com/product-info/datasheets/data/irlz44n.pdf" H 6500 3160 50  0001 L CNN
+	1    6500 3160
+	1    0    0    -1
+$EndComp
+$Comp
+L Transistor_FET:IRLZ44N Q2
+U 1 1 63FC185E
+P 7140 3820
+F 0 "Q2" H 7345 3867 50  0000 L CNN
+F 1 "IRLZ44N" H 7345 3774 50  0000 L CNN
+F 2 "Package_TO_SOT_THT:TO-220-3_Vertical" H 7390 3745 50  0001 L CIN
+F 3 "http://www.irf.com/product-info/datasheets/data/irlz44n.pdf" H 7140 3820 50  0001 L CNN
+	1    7140 3820
+	1    0    0    -1
+$EndComp
+$Comp
+L Transistor_FET:IRLZ44N Q3
+U 1 1 63FC4B32
+P 7850 4490
+F 0 "Q3" H 8055 4537 50  0000 L CNN
+F 1 "IRLZ44N" H 8055 4444 50  0000 L CNN
+F 2 "Package_TO_SOT_THT:TO-220-3_Vertical" H 8100 4415 50  0001 L CIN
+F 3 "http://www.irf.com/product-info/datasheets/data/irlz44n.pdf" H 7850 4490 50  0001 L CNN
+	1    7850 4490
+	1    0    0    -1
+$EndComp
 $EndSCHEMATC
